File: sch/ram.sch (EAGLE design)
At the start: 19 parts, among them IC1 74LS373N, IC10 74LS04N, IC11 74LS00N, IC12 74LS00N, IC13 74LS00N, IC14 74LS08N, IC15 74LS32N, IC16 74LS02N, IC4 74LS257N, IC5 74LS257N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

Commit message: Updated RAM schematics signal names.
Connections:
- net !RAMSELECT! renamed !RAM-ENABLE!
- net !REGSELECT! renamed !REG-ENABLE!
Changed lines of the file:
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@@
 </segment>
 </net>
-<net name="!REGSELECT!" class="0">
+<net name="!REG-ENABLE!" class="0">
 <segment>
 <pinref part="IC15" gate="A" pin="I1"/>
@@
 </segment>
 </net>
-<net name="!RAMSELECT!" class="0">
+<net name="!RAM-ENABLE!" class="0">
 <segment>
 <pinref part="IC1" gate="A" pin="OC"/>
